Commit message: latest dump

File: med7.urdf (robot description, URDF)
Before this commit: robot med7, 10 links, 9 joints
Links:
- removed link lbr_link_ee
- link lbr_link_0: geometry collision mesh filename=med7/collision/link_0.stl; visual mesh filename=med7/visual/link_0.dae
- link lbr_link_1: geometry collision mesh filename=med7/collision/link_1.stl; visual mesh filename=med7/visual/link_1.dae
- link lbr_link_2: geometry collision mesh filename=med7/collision/link_2.stl; visual mesh filename=med7/visual/link_2.dae
- link lbr_link_3: geometry collision mesh filename=med7/collision/link_3.stl; visual mesh filename=med7/visual/link_3.dae
- link lbr_link_4: geometry collision mesh filename=med7/collision/link_4.stl; visual mesh filename=med7/visual/link_4.dae
- link lbr_link_5: geometry collision mesh filename=med7/collision/link_5.stl; visual mesh filename=med7/visual/link_5.dae
- link lbr_link_6: geometry collision mesh filename=med7/collision/link_6.stl; visual mesh filename=med7/visual/link_6.dae
- link lbr_link_7: geometry collision mesh filename=med7/collision/link_7.stl; visual mesh filename=med7/visual/link_7.dae
Joints:
- removed joint lbr_joint_ee

Commit message: changes

File: med7.urdf (robot description, URDF)
Before this commit: robot med7, 10 links, 9 joints
Links:
- link lbr_link_0: geometry collision mesh filename=meshes/med7/collision/link_0.stl; visual mesh filename=meshes/med7/visual/link_0.dae
- link lbr_link_1: geometry collision mesh filename=meshes/med7/collision/link_1.stl; visual mesh filename=meshes/med7/visual/link_1.dae
- link lbr_link_2: geometry collision mesh filename=meshes/med7/collision/link_2.stl; visual mesh filename=meshes/med7/visual/link_2.dae
- link lbr_link_3: geometry collision mesh filename=meshes/med7/collision/link_3.stl; visual mesh filename=meshes/med7/visual/link_3.dae
- link lbr_link_4: geometry collision mesh filename=meshes/med7/collision/link_4.stl; visual mesh filename=meshes/med7/visual/link_4.dae
- link lbr_link_5: geometry collision mesh filename=meshes/med7/collision/link_5.stl; visual mesh filename=meshes/med7/visual/link_5.dae
- link lbr_link_6: geometry collision mesh filename=meshes/med7/collision/link_6.stl; visual mesh filename=meshes/med7/visual/link_6.dae
- link lbr_link_7: geometry collision mesh filename=meshes/med7/collision/link_7.stl; visual mesh filename=meshes/med7/visual/link_7.dae
